File: xadow_breakout/xadow_breakout.kicad_pcb (KiCad board)
At the start: 2 copper layers, 2 parts, among them J1 FH26W-35S-0.3SHW, J2 FH26W-35S-0.3SHW

Commit message: doc
Parts:
- added J3: microusb, mybays_connector:USB_Micro-B_Wuerth_629105150521_CircularHoles, F.Cu at (135.3, 131.2)
- added J4: Conn_01x05, Connector_PinHeader_2.54mm:PinHeader_1x05_P2.54mm_Vertical, F.Cu at (130.1, 115.9)
- added J5: Conn_01x10, Connector_PinHeader_2.54mm:PinHeader_1x10_P2.54mm_Vertical, F.Cu at (130.1, 120.5)
- added U1: LM1117-3.3, Package_TO_SOT_SMD:SOT-223-3_TabPin2, F.Cu at (116.9, 123.5)
Connections:
- net LPTE renamed LCD_TE
- net LSA0 renamed LCD_SCL
- net LSCE_B renamed LCD_CS
- net LSCK0 renamed LCD_DC
- net LSDA0 renamed LCD_SDA
- net LSRSTB renamed LCD_RST
- J1 pad 30: (no net) -> GND
- J2 pad 6: (no net) -> GND

Commit message: 20220120
Parts:
- added C1: C_Small, Capacitor_SMD:C_1210_3225Metric_Pad1.33x2.70mm_HandSolder, F.Cu at (106.0, 91.5)
- moved J4 45.5 mm to (103.6, 78.8)
- moved J5 42.1 mm to (124.3, 78.8)
- moved J2 38.8 mm to (140.0, 60.0), turned to 180 degrees
- moved J1 38.7 mm to (110.0, 60.0), turned to 180 degrees
- moved J3 37.6 mm to (125.0, 95.0)
- moved U1 31.0 mm to (113.8, 92.7)
Other:
- board outline added: 50 x 50 mm

Commit message: xadow
Parts:
- added H1: MountingHole, MountingHole:MountingHole_3.2mm_M3_ISO7380, F.Cu at (103.0, 53.0)
- added H2: MountingHole, MountingHole:MountingHole_3.2mm_M3_ISO7380, F.Cu at (147.0, 53.0)
- added H3: MountingHole, MountingHole:MountingHole_3.2mm_M3_ISO7380, F.Cu at (147.0, 97.0)
- added H4: MountingHole, MountingHole:MountingHole_3.2mm_M3_ISO7380, F.Cu at (103.0, 97.0)
- J4: value Conn_01x05 -> Conn_01x08; footprint Connector_PinHeader_2.54mm:PinHeader_1x05_P2.54mm_Vertical -> Connector_PinHeader_2.54mm:PinHeader_1x08_P2.54mm_Vertical
- moved J4 4.19 mm to (101.9, 75.0)
- moved J5 4.03 mm to (125.5, 75.0)
- moved U1 3.05 mm to (115.4, 90.1)
- moved J1 2.00 mm to (110.0, 62.0)
- moved J2 2.00 mm to (140.0, 62.0)
- moved C1 1.98 mm to (108.0, 91.2), turned to 270 degrees
- moved J3 0.50 mm to (125.0, 95.5)
Connections:
- J4 pad 1: CTP_SDA -> +3V3
- J4 pad 2: CTP_SCL -> +2V8
- J4 pad 3: CTP_EINT -> GND
- J4 pad 4: CTP_RST -> CTP_SDA
- J4 pad 5: GND -> CTP_SCL
- J5 pad 1: (no net) -> +3V3
- J5 pad 2: (no net) -> GND
Routing:
- net LCD_SCL: track 0.00 -> 81.0 mm, vias 0 -> 3
- net PWM_BACKLIGHT: track 0.00 -> 78.3 mm
- net LCD_RST: track 0.00 -> 75.4 mm, vias 0 -> 1
- net CTP_SDA: track 0.00 -> 70.2 mm, vias 0 -> 2
- net CTP_RST: track 0.00 -> 65.3 mm, vias 0 -> 1
- net CTP_SCL: track 0.00 -> 63.7 mm
- net LCD_CS: track 0.00 -> 63.3 mm, vias 0 -> 1
- net +2V8: track 0.00 -> 56.5 mm, vias 0 -> 1
- net LCD_DC: track 0.00 -> 54.4 mm, vias 0 -> 1
- net +3V3: track 0.00 -> 53.6 mm, vias 0 -> 2
- net LCD_SDA: track 0.00 -> 52.1 mm, vias 0 -> 2
- net LCD_TE: track 0.00 -> 44.9 mm, vias 0 -> 1
- net CTP_EINT: track 0.00 -> 41.4 mm, vias 0 -> 1
- net GND: track 0.00 -> 38.8 mm, vias 0 -> 8
- net Net-(J3-Pad1): track 0.00 -> 10.0 mm
- added copper zone on In2.Cu, net +3V3
- added copper zone on In1.Cu, net GND
Other:
- copper layers 2 -> 4
- board text added: "2V8"
- board text added: "3V3"
- board text added: "CS"
- board text added: "DC"
- board text added: "GND"
- board text added: "INT"
- board text added: "LCD"
- board text added: "PWM"
- board text added: "RST"
- board text added: "SCL"
- board text added: "SDA"
- board text added: "TE"
- board text added: "TOUCH"
- board text added: "Xadow 1.54"
