File: xadow_breakout/xadow_breakout.sch (KiCad schematic (older format))
At the start: 2 parts, among them J1 FH26W-35S-0.3SHW, J2 FH26W-35S-0.3SHW

Commit message: doc
Parts:
- added J3: microusb, mybays_connector:USB_Micro-B_Wuerth_629105150521_CircularHoles, symbol mybays_connector:microusb
- added J4: Conn_01x05, Connector_PinHeader_2.54mm:PinHeader_1x05_P2.54mm_Vertical, symbol Connector_Generic:Conn_01x05
- added J5: Conn_01x10, Connector_PinHeader_2.54mm:PinHeader_1x10_P2.54mm_Vertical, symbol Connector_Generic:Conn_01x10
- added U1: LM1117-3.3, Package_TO_SOT_SMD:SOT-223-3_TabPin2, symbol Regulator_Linear:LM1117-3.3
Connections:
- net labels added: LCD_CS, LCD_DC, LCD_RST, LCD_SCL, LCD_SDA, LCD_TE
- net labels removed: LPTE, LSA0, LSCE_B, LSCK0, LSDA0, LSRSTB
- wire segments 74 -> 96
Other:
- moved on the sheet: J1, J2

Commit message: 20220120
Parts:
- added C1: C_Small, Capacitor_SMD:C_1210_3225Metric_Pad1.33x2.70mm_HandSolder, symbol Device:C_Small
Connections:
- wire segments 96 -> 101

Commit message: xadow
Parts:
- added H1, H2, H3, H4: MountingHole, MountingHole:MountingHole_3.2mm_M3_ISO7380, symbol Mechanical:MountingHole
- J4: value Conn_01x05 -> Conn_01x08; footprint Connector_PinHeader_2.54mm:PinHeader_1x05_P2.54mm_Vertical -> Connector_PinHeader_2.54mm:PinHeader_1x08_P2.54mm_Vertical; symbol Connector_Generic:Conn_01x05 -> Connector_Generic:Conn_01x08
Connections:
- wire segments 101 -> 104
Changed lines of the file:
@@
 	1100 6500 1800 6500
 $Comp
-L Connector_Generic:Conn_01x05 J4
+L Connector_Generic:Conn_01x08 J4
 U 1 1 61E95C9B
 P 3650 5100
 F 0 "J4" H 3730 5142 50  0000 L CNN
-F 1 "Conn_01x05" H 3730 5051 50  0000 L CNN
-F 2 "Connector_PinHeader_2.54mm:PinHeader_1x05_P2.54mm_Vertical" H 3650 5100 50  0001 C CNN
+F 1 "Conn_01x08" H 3730 5051 50  0000 L CNN
+F 2 "Connector_PinHeader_2.54mm:PinHeader_1x08_P2.54mm_Vertical" H 3650 5100 50  0001 C CNN
 F 3 "~" H 3650 5100 50  0001 C CNN
 	1    3650 5100
@@
 L power:GND #PWR0118
 U 1 1 61EBCCCA
-P 3400 5300
-F 0 "#PWR0118" H 3400 5050 50  0001 C CNN
-F 1 "GND" H 3405 5127 50  0000 C CNN
-F 2 "" H 3400 5300 50  0001 C CNN
-F 3 "" H 3400 5300 50  0001 C CNN
-	1    3400 5300
+P 3400 5500
+F 0 "#PWR0118" H 3400 5250 50  0001 C CNN
+F 1 "GND" H 3405 5327 50  0000 C CNN
+F 2 "" H 3400 5500 50  0001 C CNN
+F 3 "" H 3400 5500 50  0001 C CNN
+	1    3400 5500
 	0    1    1    0
 $EndComp
+Text GLabel 3400 5400 0    50   Input ~ 0
+CTP_RST
+Text GLabel 3400 5300 0    50   Input ~ 0
+CTP_EINT
+Text GLabel 3400 5100 0    50   Input ~ 0
+CTP_SDA
 Text GLabel 3400 5200 0    50   Input ~ 0
-CTP_RST
-Text GLabel 3400 5100 0    50   Input ~ 0
-CTP_EINT
-Text GLabel 3400 4900 0    50   Input ~ 0
-CTP_SDA
-Text GLabel 3400 5000 0    50   Input ~ 0
 CTP_SCL
 $Comp
@@
 Wire Wire Line
 	2100 6850 2100 6900
+$Comp
+L power:GND #PWR0120
+U 1 1 61F23712
+P 6300 4650
+F 0 "#PWR0120" H 6300 4400 50  0001 C CNN
+F 1 "GND" H 6305 4477 50  0000 C CNN
+F 2 "" H 6300 4650 50  0001 C CNN
+F 3 "" H 6300 4650 50  0001 C CNN
+	1    6300 4650
+	0    1    1    0
+$EndComp
+$Comp
+L power:+3V3 #PWR0121
+U 1 1 61F23B64
+P 6300 4550
+F 0 "#PWR0121" H 6300 4400 50  0001 C CNN
+F 1 "+3V3" V 6315 4678 50  0000 L CNN
+F 2 "" H 6300 4550 50  0001 C CNN
+F 3 "" H 6300 4550 50  0001 C CNN
+	1    6300 4550
+	0    -1   -1   0
+$EndComp
+Wire Wire Line
+	3400 5400 3450 5400
+Wire Wire Line
+	3400 5500 3450 5500
+Wire Wire Line
+	3400 4800 3450 4800
+$Comp
+L power:GND #PWR0122
+U 1 1 61F3B110
+P 3400 5000
+F 0 "#PWR0122" H 3400 4750 50  0001 C CNN
+F 1 "GND" H 3405 4827 50  0000 C CNN
+F 2 "" H 3400 5000 50  0001 C CNN
+F 3 "" H 3400 5000 50  0001 C CNN
+	1    3400 5000
+	0    1    1    0
+$EndComp
+$Comp
+L power:+2V8 #PWR0123
+U 1 1 61F3B455
+P 3400 4900
+F 0 "#PWR0123" H 3400 4750 50  0001 C CNN
+F 1 "+2V8" V 3415 5028 50  0000 L CNN
+F 2 "" H 3400 4900 50  0001 C CNN
+F 3 "" H 3400 4900 50  0001 C CNN
+	1    3400 4900
+	0    -1   -1   0
+$EndComp
+$Comp
+L power:+3V3 #PWR0124
+U 1 1 61F3B9BC
+P 3400 4800
+F 0 "#PWR0124" H 3400 4650 50  0001 C CNN
+F 1 "+3V3" V 3415 4928 50  0000 L CNN
+F 2 "" H 3400 4800 50  0001 C CNN
+F 3 "" H 3400 4800 50  0001 C CNN
+	1    3400 4800
+	0    -1   -1   0
+$EndComp
+$Comp
+L Mechanical:MountingHole H1
+U 1 1 61F4C5A9
+P 10350 5250
+F 0 "H1" H 10450 5296 50  0000 L CNN
+F 1 "MountingHole" H 10450 5205 50  0000 L CNN
+F 2 "MountingHole:MountingHole_3.2mm_M3_ISO7380" H 10350 5250 50  0001 C CNN
+F 3 "~" H 10350 5250 50  0001 C CNN
+	1    10350 5250
+	1    0    0    -1
+$EndComp
+$Comp
+L Mechanical:MountingHole H2
+U 1 1 61F4C8CD
+P 10350 5400
+F 0 "H2" H 10450 5446 50  0000 L CNN
+F 1 "MountingHole" H 10450 5355 50  0000 L CNN
+F 2 "MountingHole:MountingHole_3.2mm_M3_ISO7380" H 10350 5400 50  0001 C CNN
+F 3 "~" H 10350 5400 50  0001 C CNN
+	1    10350 5400
+	1    0    0    -1
+$EndComp
+$Comp
+L Mechanical:MountingHole H3
+U 1 1 61F4CBAB
+P 10350 5550
+F 0 "H3" H 10450 5596 50  0000 L CNN
+F 1 "MountingHole" H 10450 5505 50  0000 L CNN
+F 2 "MountingHole:MountingHole_3.2mm_M3_ISO7380" H 10350 5550 50  0001 C CNN
+F 3 "~" H 10350 5550 50  0001 C CNN
+	1    10350 5550
+	1    0    0    -1
+$EndComp
+$Comp
+L Mechanical:MountingHole H4
+U 1 1 61F4CDE8
+P 10350 5700
+F 0 "H4" H 10450 5746 50  0000 L CNN
+F 1 "MountingHole" H 10450 5655 50  0000 L CNN
+F 2 "MountingHole:MountingHole_3.2mm_M3_ISO7380" H 10350 5700 50  0001 C CNN
+F 3 "~" H 10350 5700 50  0001 C CNN
+	1    10350 5700
+	1    0    0    -1
+$EndComp
 $EndSCHEMATC
